Commit message: Update with fisheye files

File: my_robot_description/urdf/rig_prototype_2.urdf (robot description, URDF)
Before this commit: robot my_robot, 17 links, 16 joints
Joints:
- joint camera_joint: axis 0 0 0 -> 5 5 20; origin xyz=1.1 5.1 4 rpy=0 -0.785 -1.570796327 -> xyz=1.1 5.1 4 rpy=0 0.785 1.570796327
